File: keyboard/keyboard.kicad_pcb (KiCad board)
At the start: 2 copper layers, 319.9 x 104.8 mm, 130 parts, among them SW1 `, SW10 0, SW11 -, SW12 =, SW13 Esc, SW14 Tab, SW15 Q, SW16 W, SW17 E, SW18 R, SW19 T, SW2 1, SW20 Y, SW21 U, SW22 I, SW23 O, SW24 P, SW25 [, SW26 ], SW27 \, SW28 Home, SW29 Hyper, SW3 3, SW30 A, SW31 S, SW32 D, SW33 F, SW34 G, SW35 H, SW36 J, SW37 K, SW38 L, SW39 ;, SW4 4, SW40 ', SW41 Backspace, SW42 Insert, SW43 LShift, SW44 Z, SW45 X, SW46 C, SW47 V, SW48 B, SW49 N, SW5 5, SW51 M, SW52 ,, SW53 ., SW54 /, SW55 Enter, SW56 PageUp, SW57 LCtrl, SW58 Win, SW59 LAlt, SW6 6, SW60 Space, SW61 RAlt, SW62 Menu, SW63 RCtrl, SW64 Print, SW65 2, SW7 7, SW8 8, SW9 9, U1 Elite-C

Commit message: completed pcb layout
Parts:
- removed D50: D, Keebio-Parts:D_0805
- added REF**: MountingHole_3.5mm, MountingHole:MountingHole_3.5mm, F.Cu at (335.8, 24.6)
- added REF**: MountingHole_3.5mm, MountingHole:MountingHole_3.5mm, F.Cu at (335.8, 118.3)
- added REF**: MountingHole_3.5mm, MountingHole:MountingHole_3.5mm, F.Cu at (21.4, 118.3)
- added REF**: MountingHole_3.5mm, MountingHole:MountingHole_3.5mm, F.Cu at (21.4, 24.6)
- D1, D10, D11, D12, D13, D14, D15, D16, D17, D18, D19, D2, D20, D21, D22, D23, D24, D25, D26, D27, D28, D29, D3, D30, D31, D32, D33, D34, D35, D36, D37, D38, D39, D4, D40, D41, D42, D43, D44, D45, D46, D47, D48, D49, D5, D51, D52, D53, D54, D55, D56, D57, D58, D59, D6, D60, D61, D62, D63, D64, D65, D7, D8, D9: moved to B.Cu
- moved D56 558.9 mm to (330.2, 85.7), turned to 270 degrees
- moved D64 557.7 mm to (330.2, 104.8), turned to 270 degrees
- moved D42 538.0 mm to (330.2, 66.7), turned to 270 degrees
- moved D13 537.0 mm to (330.2, 28.6), turned to 270 degrees
- moved D28 532.3 mm to (330.2, 47.6), turned to 270 degrees
- moved D55 522.4 mm to (288.9, 85.7), turned to 270 degrees
- moved D63 519.0 mm to (286.5, 104.8), turned to 270 degrees
- moved D41 513.6 mm to (296.1, 66.7), turned to 270 degrees
- moved D62 504.6 mm to (267.5, 104.8), turned to 270 degrees
- moved D54 496.2 mm to (258.0, 85.7), turned to 270 degrees
- moved D27 494.1 mm to (296.1, 47.6), turned to 270 degrees
- moved D12 490.0 mm to (286.5, 28.6), turned to 270 degrees
- moved D11 485.6 mm to (267.5, 28.6), turned to 270 degrees
- moved D40 480.8 mm to (267.5, 66.7), turned to 270 degrees
- moved D61 480.8 mm to (248.4, 104.8), turned to 270 degrees
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Connections:
- D10 pad 1: Net-(D10-Pad1) -> Row0
- D11 pad 1: Net-(D10-Pad2) -> Row0
- D12 pad 1: Net-(D11-Pad2) -> Row0
- D13 pad 1: Net-(D12-Pad2) -> Row0
- D15 pad 1: Net-(D14-Pad2) -> Row1
- D16 pad 1: Net-(D15-Pad2) -> Row1
- D17 pad 1: Net-(D16-Pad2) -> Row1
- D18 pad 1: Net-(D17-Pad2) -> Row1
- D19 pad 1: Net-(D18-Pad2) -> Row1
- D2 pad 1: Net-(D1-Pad2) -> Row0
- D20 pad 1: Net-(D19-Pad2) -> Row1
- D21 pad 1: Net-(D20-Pad2) -> Row1
- D22 pad 1: Net-(D21-Pad2) -> Row1
- D23 pad 1: Net-(D22-Pad2) -> Row1
- D24 pad 1: Net-(D23-Pad2) -> Row1
- D25 pad 1: Net-(D24-Pad2) -> Row1
- D26 pad 1: Net-(D25-Pad2) -> Row1
- D27 pad 1: Net-(D26-Pad2) -> Row1
- D28 pad 1: Net-(D27-Pad2) -> Row1
- D3 pad 1: Net-(D2-Pad2) -> Row0
- D30 pad 1: Net-(D29-Pad2) -> Row2
- D31 pad 1: Net-(D30-Pad2) -> Row2
- D32 pad 1: Net-(D31-Pad2) -> Row2
- D33 pad 1: Net-(D32-Pad2) -> Row2
- D34 pad 1: Net-(D33-Pad2) -> Row2
- D35 pad 1: Net-(D34-Pad2) -> Row2
- D36 pad 1: Net-(D35-Pad2) -> Row2
- D37 pad 1: Net-(D36-Pad2) -> Row2
- D38 pad 1: Net-(D37-Pad2) -> Row2
- D39 pad 1: Net-(D38-Pad2) -> Row2
- D4 pad 1: Net-(D4-Pad1) -> Row0
- D40 pad 1: Net-(D39-Pad2) -> Row2
- D41 pad 1: Net-(D40-Pad2) -> Row2
- D42 pad 1: Net-(D41-Pad2) -> Row2
- D44 pad 1: Net-(D43-Pad2) -> Row3
- D45 pad 1: Net-(D44-Pad2) -> Row3
- D46 pad 1: Net-(D45-Pad2) -> Row3
- D47 pad 1: Net-(D46-Pad2) -> Row3
- D48 pad 1: Net-(D47-Pad2) -> Row3
- D49 pad 1: Net-(D48-Pad2) -> Row3
- D5 pad 1: Net-(D4-Pad2) -> Row0
- D51 pad 1: Net-(D49-Pad2) -> Row3
- D52 pad 1: Net-(D51-Pad2) -> Row3
- D53 pad 1: Net-(D52-Pad2) -> Row3
- D54 pad 1: Net-(D53-Pad2) -> Row3
- D55 pad 1: Net-(D54-Pad2) -> Row3
- D56 pad 1: Net-(D55-Pad2) -> Row3
- D58 pad 1: Net-(D57-Pad2) -> Row4
- D59 pad 1: Net-(D58-Pad2) -> Row4
- D6 pad 1: Net-(D5-Pad2) -> Row0
- D60 pad 1: Net-(D59-Pad2) -> Row4
- D61 pad 1: Net-(D60-Pad2) -> Row4
- D62 pad 1: Net-(D61-Pad2) -> Row4
- D63 pad 1: Net-(D62-Pad2) -> Row4
- D64 pad 1: Net-(D63-Pad2) -> Row4
- D65 pad 1: Net-(D3-Pad2) -> Row0
- D65 pad 2: Net-(D4-Pad1) -> Net-(D65-Pad2)
- D7 pad 1: Net-(D6-Pad2) -> Row0
- D8 pad 1: Net-(D7-Pad2) -> Row0
- D9 pad 1: Net-(D8-Pad2) -> Row0
- D9 pad 2: Net-(D10-Pad1) -> Net-(D9-Pad2)
- SW13 pad 2: Col15 -> Col14
- SW28 pad 2: Col15 -> Col14
- SW3 pad 1: Net-(D4-Pad1) -> Net-(D65-Pad2)
- SW42 pad 2: Col15 -> Col14
- SW56 pad 2: Col15 -> Col14
- SW64 pad 2: Col15 -> Col14
- SW9 pad 1: Net-(D10-Pad1) -> Net-(D9-Pad2)
- U1 pad 10: Col5 -> Col2
- U1 pad 11: Col6 -> Col1
- U1 pad 12: Col7 -> Col0
- U1 pad 14: Col15 -> Col8
- U1 pad 15: Col13 -> Col9
- U1 pad 16: Col12 -> Col10
- U1 pad 18: Col10 -> Col12
- U1 pad 19: Col9 -> Col13
- U1 pad 20: Col8 -> Col14
- U1 pad 5: Col0 -> Col7
- U1 pad 6: Col1 -> Col6
- U1 pad 7: Col2 -> Col5
- U1 pad 8: Col3 -> Col4
- U1 pad 9: Col4 -> Col3
Routing:
- net Col14: track 0.00 -> 397.5 mm, vias 0 -> 3
- net Row0: track 0.00 -> 373.6 mm, vias 0 -> 2
- net Row1: track 0.00 -> 369.5 mm
- net Col12: track 0.00 -> 353.0 mm, vias 0 -> 3
- net Row2: track 0.00 -> 341.8 mm
- net Row3: track 0.00 -> 341.7 mm
- net Row4: track 0.00 -> 335.9 mm
- net Col13: track 0.00 -> 331.1 mm, vias 0 -> 7
- net Col11: track 0.00 -> 321.8 mm, vias 0 -> 3
- net Col10: track 0.00 -> 290.4 mm, vias 0 -> 3
- net Col9: track 0.00 -> 268.9 mm, vias 0 -> 3
- net Col7: track 0.00 -> 247.6 mm, vias 0 -> 3
- net Col8: track 0.00 -> 245.8 mm, vias 0 -> 3
- net Col5: track 0.00 -> 237.0 mm, vias 0 -> 3
- net Col6: track 0.00 -> 226.7 mm, vias 0 -> 3
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Other:
- board size 319.9 x 104.8 mm -> 325.4 x 104.8 mm
- rule via_min_size: 0.4 -> 0.2
